Commit message: Added LiDAR and fixed robot init bug
Gazebo's URDF spawner crashes when it inserts robot before env is ready.

- Added configurable node_start_delay to launch file to cater for larger
envs.
- Added LiDAR onto robot and regenerated champ.urdf.

File: champ_description/urdf/accessories.urdf.xacro (robot description, xacro)
@@ -43,8 +43,10 @@
             <child link="imu_link" />
         </joint>
-        <!-- <xacro:include filename="$(find velodyne_description)/urdf/VLP-16.urdf.xacro"/>
-        <xacro:VLP-16 parent="${base_name}" name="velodyne" topic="velodyne_points" hz="10" samples="1024" gpu="false" lasers="16" max_range="100">
+        <xacro:include filename="$(find velodyne_description)/urdf/VLP-16.urdf.xacro"/>
+        <!-- <xacro:VLP-16 parent="${base_name}" name="velodyne" topic="velodyne_points" hz="10" samples="1024" gpu="false" lasers="16" max_range="100"> -->
+        <xacro:VLP-16 parent="${base_name}" name="velodyne" topic="velodyne_points" hz="10" samples="350" gpu="false" min_range="0.001">
             <origin xyz="0 0 ${base_height / 2}" rpy="0 0 0" />
         </xacro:VLP-16>
+        <!--
         <xacro:include filename="$(find champ_arm_description)/urdf/champ_arm.urdf.xacro" />
         <xacro:champ_arm parent="${base_name}">

File: champ_description/urdf/champ.urdf (robot description, URDF)
Before this commit: robot champ, 29 links, 28 joints
Links:
- added link velodyne, mass 0.01; visual mesh filename=package://velodyne_description/meshes/VLP16_scan.dae
- added link velodyne_base_link, mass 0.83; collision cylinder length=0.0717 radius=0.0516; visual mesh filename=package://velodyne_description/meshes/VLP16_base_1.dae
Joints:
- added joint velodyne_base_mount_joint: type fixed, parent base_link, child velodyne_base_link, origin xyz=0 0 0.065 rpy=0 0 0
- added joint velodyne_base_scan_joint: type fixed, parent velodyne_base_link, child velodyne, origin xyz=0 0 0.0377 rpy=0 0 0
- joint camera_depth_optical_joint: origin xyz=0 0 0 rpy=-1.57079632679 0.0 -1.57079632679 -> xyz=0 0 0 rpy=-1.5707963267948966 0.0 -1.5707963267948966
- joint camera_rgb_optical_joint: origin xyz=0 0 0 rpy=-1.57079632679 0.0 -1.57079632679 -> xyz=0 0 0 rpy=-1.5707963267948966 0.0 -1.5707963267948966
- joint hokuyo_joint: origin xyz=0.0 0.0 0.105 rpy=0 0 0 -> xyz=0.0 0.0 0.10500000000000001 rpy=0 0 0
- joint lf_hip_joint: limit lower=-3.14159265359 upper=3.14159265359 effort=25 velocity=1.5 -> lower=-3.141592653589793 upper=3.141592653589793 effort=25 velocity=1.5
- joint lf_lower_leg_joint: limit lower=-3.14159265359 upper=3.14159265359 effort=25 velocity=1.5 -> lower=-3.141592653589793 upper=3.141592653589793 effort=25 velocity=1.5
- joint lf_upper_leg_joint: limit lower=-3.14159265359 upper=3.14159265359 effort=25 velocity=1.5 -> lower=-3.141592653589793 upper=3.141592653589793 effort=25 velocity=1.5
- joint lh_hip_joint: limit lower=-3.14159265359 upper=3.14159265359 effort=25 velocity=1.5 -> lower=-3.141592653589793 upper=3.141592653589793 effort=25 velocity=1.5
- joint lh_lower_leg_joint: limit lower=-3.14159265359 upper=3.14159265359 effort=25 velocity=1.5 -> lower=-3.141592653589793 upper=3.141592653589793 effort=25 velocity=1.5
- joint lh_upper_leg_joint: limit lower=-3.14159265359 upper=3.14159265359 effort=25 velocity=1.5 -> lower=-3.141592653589793 upper=3.141592653589793 effort=25 velocity=1.5
- joint rf_hip_joint: limit lower=-3.14159265359 upper=3.14159265359 effort=25 velocity=1.5 -> lower=-3.141592653589793 upper=3.141592653589793 effort=25 velocity=1.5
- joint rf_lower_leg_joint: limit lower=-3.14159265359 upper=3.14159265359 effort=25 velocity=1.5 -> lower=-3.141592653589793 upper=3.141592653589793 effort=25 velocity=1.5
- joint rf_upper_leg_joint: limit lower=-3.14159265359 upper=3.14159265359 effort=25 velocity=1.5 -> lower=-3.141592653589793 upper=3.141592653589793 effort=25 velocity=1.5
- joint rh_hip_joint: limit lower=-3.14159265359 upper=3.14159265359 effort=25 velocity=1.5 -> lower=-3.141592653589793 upper=3.141592653589793 effort=25 velocity=1.5
- joint rh_lower_leg_joint: limit lower=-3.14159265359 upper=3.14159265359 effort=25 velocity=1.5 -> lower=-3.141592653589793 upper=3.141592653589793 effort=25 velocity=1.5
- joint rh_upper_leg_joint: limit lower=-3.14159265359 upper=3.14159265359 effort=25 velocity=1.5 -> lower=-3.141592653589793 upper=3.141592653589793 effort=25 velocity=1.5
